File: PCB/v0.1/esp32_display/pwr.kicad_sch (KiCad schematic)
At the start: 12 parts, among them U2 MAX1821

Commit message: Smaller footprint, no housing, right angle buttons
Parts:
- removed C12: 0.1pF, Capacitor_SMD:C_0603_1608Metric_Pad1.08x0.95mm_HandSolder, symbol Device:C
- C9: value 0.047uF -> 47nF
Other:
- note removed: "Can be omitted due to use of ceramic capacitors."
Changed lines of the file:
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@@
   (junction (at 55.88 80.01) (diameter 0) (color 0 0 0 0)
   )
-  (junction (at 124.46 106.68) (diameter 0) (color 0 0 0 0)
-  )
   (junction (at 81.28 80.01) (diameter 0) (color 0 0 0 0)
   )
@@
   (junction (at 152.4 80.01) (diameter 0) (color 0 0 0 0)
   )
-  (junction (at 124.46 123.19) (diameter 0) (color 0 0 0 0)
-  )
-  (wire (pts (xy 139.7 106.68) (xy 124.46 106.68))
-    (stroke (width 0) (type default) (color 0 0 0 0))
-  )
   (wire (pts (xy 152.4 80.01) (xy 152.4 88.9))
     (stroke (width 0) (type default) (color 0 0 0 0))
@@
     (stroke (width 0) (type default) (color 0 0 0 0))
   )
-  (wire (pts (xy 139.7 119.38) (xy 139.7 123.19))
-    (stroke (width 0) (type default) (color 0 0 0 0))
-  )
   (wire (pts (xy 58.42 178.435) (xy 58.42 180.34))
     (stroke (width 0) (type default) (color 0 0 0 0))
@@
     (stroke (width 0) (type default) (color 0 0 0 0))
   )
-  (wire (pts (xy 139.7 123.19) (xy 124.46 123.19))
-    (stroke (width 0) (type default) (color 0 0 0 0))
-  )
   (wire (pts (xy 119.38 80.01) (xy 116.84 80.01))
     (stroke (width 0) (type default) (color 0 0 0 0))
@@
   )
   (wire (pts (xy 130.81 87.63) (xy 116.84 87.63))
-    (stroke (width 0) (type default) (color 0 0 0 0))
-  )
-  (wire (pts (xy 139.7 111.76) (xy 139.7 106.68))
     (stroke (width 0) (type default) (color 0 0 0 0))
   )
@@
   )
   (text "For calculation see MAX1821.ods file" (at 129.54 127 0)
-    (effects (font (size 1.27 1.27)) (justify left bottom))
-  )
-  (text "Can be omitted due to use of ceramic capacitors." (at 140.97 120.65 0)
     (effects (font (size 1.27 1.27)) (justify left bottom))
   )
@@
       (effects (font (size 1.27 1.27)) (justify left))
     )
-    (property "Value" "0.047uF" (id 1) (at 80.391 114.173 0)
+    (property "Value" "47nF" (id 1) (at 80.391 114.173 0)
       (effects (font (size 1.27 1.27)) (justify left))
     )
@@
     (pin "1")
   )
-  (symbol (lib_id "Device:C") (at 139.7 115.57 0) (unit 1)
-    (in_bom yes) (on_board yes)
-    (property "Reference" "C12" (id 0) (at 142.621 114.4016 0)
-      (effects (font (size 1.27 1.27)) (justify left))
-    )
-    (property "Value" "0.1pF" (id 1) (at 142.621 116.713 0)
-      (effects (font (size 1.27 1.27)) (justify left))
-    )
-    (property "Footprint" "Capacitor_SMD:C_0603_1608Metric_Pad1.08x0.95mm_HandSolder" (id 2) (at 140.6652 119.38 0)
-      (effects (font (size 1.27 1.27)) hide)
-    )
-    (property "Datasheet" "~" (id 3) (at 139.7 115.57 0)
-      (effects (font (size 1.27 1.27)) hide)
-    )
-    (pin "1")
-    (pin "2")
-  )
   (symbol (lib_id "Device:C") (at 142.24 83.82 0) (unit 1)

Commit message: Add serial resistors to SPI lines (PCB not finished)
Still missing placment of RC filters.
Parts:
- renumbered C9 to C10, C10 to C11, C11 to C12, C7 to C8, C8 to C9, R5 to R18, R6 to R19, R7 to R20
Changed lines of the file:
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@@
   (symbol (lib_id "Device:C") (at 55.88 85.09 0) (unit 1)
     (in_bom yes) (on_board yes)
-    (property "Reference" "C7" (id 0) (at 58.801 83.9216 0)
+    (property "Reference" "C8" (id 0) (at 58.801 83.9216 0)
       (effects (font (size 1.27 1.27)) (justify left))
     )
@@
   (symbol (lib_id "power:GND") (at 99.06 115.57 0) (unit 1)
     (in_bom yes) (on_board yes)
-    (property "Reference" "#PWR027" (id 0) (at 99.06 121.92 0)
+    (property "Reference" "#PWR028" (id 0) (at 99.06 121.92 0)
       (effects (font (size 1.27 1.27)) hide)
     )
@@
   (symbol (lib_id "power:GND") (at 105.41 115.57 0) (unit 1)
     (in_bom yes) (on_board yes)
-    (property "Reference" "#PWR028" (id 0) (at 105.41 121.92 0)
+    (property "Reference" "#PWR029" (id 0) (at 105.41 121.92 0)
       (effects (font (size 1.27 1.27)) hide)
     )
@@
   (symbol (lib_id "Device:C") (at 77.47 113.03 0) (unit 1)
     (in_bom yes) (on_board yes)
-    (property "Reference" "C9" (id 0) (at 80.391 111.8616 0)
+    (property "Reference" "C10" (id 0) (at 80.391 111.8616 0)
       (effects (font (size 1.27 1.27)) (justify left))
     )
@@
   (symbol (lib_id "Device:C") (at 124.46 119.38 0) (unit 1)
     (in_bom yes) (on_board yes)
-    (property "Reference" "C10" (id 0) (at 127.381 118.2116 0)
+    (property "Reference" "C11" (id 0) (at 127.381 118.2116 0)
       (effects (font (size 1.27 1.27)) (justify left))
     )
@@
   (symbol (lib_id "Device:R") (at 124.46 111.76 0) (unit 1)
     (in_bom yes) (on_board yes)
-    (property "Reference" "R5" (id 0) (at 126.238 110.5916 0)
+    (property "Reference" "R18" (id 0) (at 126.238 110.5916 0)
       (effects (font (size 1.27 1.27)) (justify left))
     )
@@
   (symbol (lib_id "power:GND") (at 77.47 116.84 0) (unit 1)
     (in_bom yes) (on_board yes)
-    (property "Reference" "#PWR025" (id 0) (at 77.47 123.19 0)
+    (property "Reference" "#PWR026" (id 0) (at 77.47 123.19 0)
       (effects (font (size 1.27 1.27)) hide)
     )
@@
   (symbol (lib_id "power:GND") (at 124.46 123.19 0) (unit 1)
     (in_bom yes) (on_board yes)
-    (property "Reference" "#PWR029" (id 0) (at 124.46 129.54 0)
+    (property "Reference" "#PWR030" (id 0) (at 124.46 129.54 0)
       (effects (font (size 1.27 1.27)) hide)
     )
@@
   (symbol (lib_id "Device:C") (at 69.85 85.09 0) (unit 1)
     (in_bom yes) (on_board yes)
-    (property "Reference" "C8" (id 0) (at 72.771 83.9216 0)
+    (property "Reference" "C9" (id 0) (at 72.771 83.9216 0)
       (effects (font (size 1.27 1.27)) (justify left))
     )
@@
   (symbol (lib_id "Device:C") (at 130.81 83.82 0) (unit 1)
     (in_bom yes) (on_board yes)
-    (property "Reference" "C11" (id 0) (at 133.731 82.6516 0)
+    (property "Reference" "C12" (id 0) (at 133.731 82.6516 0)
       (effects (font (size 1.27 1.27)) (justify left))
     )
@@
   (symbol (lib_id "Device:R") (at 152.4 92.71 0) (unit 1)
     (in_bom yes) (on_board yes)
-    (property "Reference" "R6" (id 0) (at 154.178 91.5416 0)
+    (property "Reference" "R19" (id 0) (at 154.178 91.5416 0)
       (effects (font (size 1.27 1.27)) (justify left))
     )
@@
   (symbol (lib_id "Device:R") (at 152.4 100.33 0) (unit 1)
     (in_bom yes) (on_board yes)
-    (property "Reference" "R7" (id 0) (at 154.178 99.1616 0)
+    (property "Reference" "R20" (id 0) (at 154.178 99.1616 0)
       (effects (font (size 1.27 1.27)) (justify left))
     )
@@
   (symbol (lib_id "power:GND") (at 152.4 104.14 0) (unit 1)
     (in_bom yes) (on_board yes)
-    (property "Reference" "#PWR031" (id 0) (at 152.4 110.49 0)
+    (property "Reference" "#PWR032" (id 0) (at 152.4 110.49 0)
       (effects (font (size 1.27 1.27)) hide)
     )
@@
   (symbol (lib_id "power:GND") (at 86.36 96.52 0) (unit 1)
     (in_bom yes) (on_board yes)
-    (property "Reference" "#PWR026" (id 0) (at 86.36 102.87 0)
+    (property "Reference" "#PWR027" (id 0) (at 86.36 102.87 0)
       (effects (font (size 1.27 1.27)) hide)
     )
@@
   (symbol (lib_id "power:GNDPWR") (at 69.85 88.9 0) (unit 1)
     (in_bom yes) (on_board yes) (fields_autoplaced)
-    (property "Reference" "#PWR0102" (id 0) (at 69.85 93.98 0)
+    (property "Reference" "#PWR025" (id 0) (at 69.85 93.98 0)
       (effects (font (size 1.27 1.27)) hide)
     )
@@
   (symbol (lib_id "power:GNDPWR") (at 49.53 180.34 0) (unit 1)
     (in_bom yes) (on_board yes) (fields_autoplaced)
-    (property "Reference" "#PWR0103" (id 0) (at 49.53 185.42 0)
+    (property "Reference" "#PWR023" (id 0) (at 49.53 185.42 0)
       (effects (font (size 1.27 1.27)) hide)
     )
@@
   (symbol (lib_id "power:GND") (at 58.42 180.34 0) (unit 1)
     (in_bom yes) (on_board yes) (fields_autoplaced)
-    (property "Reference" "#PWR0104" (id 0) (at 58.42 186.69 0)
+    (property "Reference" "#PWR024" (id 0) (at 58.42 186.69 0)
       (effects (font (size 1.27 1.27)) hide)
     )
@@
   (symbol (lib_id "power:GNDPWR") (at 130.81 87.63 0) (unit 1)
     (in_bom yes) (on_board yes) (fields_autoplaced)
-    (property "Reference" "#PWR0101" (id 0) (at 130.81 92.71 0)
-      (effects (font (size 1.27 1.27)) hide)
-    )
+    (property "Reference" "#PWR031" (id 0) (at 130.81 92.71 0)
+      (effects (font (size 1.27 1.27)) hide)
+    )
