File: Board/v0.1/display.kicad_sch (KiCad schematic)
At the start: 6 parts, among them U3 Display_ILI9341

Commit message: Clean schematics (add date and revision...)
Other:
- company: (none) -> Bzgec
- title: (none) -> Display
Changed lines of the file:
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@@
 (kicad_sch (version 20211123) (generator eeschema)
   (paper "A4")
+  (title_block
+    (title "Display")
+    (date "2022/01/06")
+    (rev "v0.1")
+    (company "Bzgec")
+  )
   (bus_alias "DISP_CONN" (members "SPI_MISO" "SPI_MOSI" "SPI_CLK" "SPI_CS" "DC" "RST" "BCKL"))
   (junction (at 99.06 30.48) (diameter 0) (color 0 0 0 0)
@@
   (symbol (lib_id "power:+3.3V") (at 99.06 30.48 0) (unit 1)
     (in_bom yes) (on_board yes) (fields_autoplaced)
-    (property "Reference" "#PWR033" (id 0) (at 99.06 34.29 0)
+    (property "Reference" "#PWR032" (id 0) (at 99.06 34.29 0)
       (effects (font (size 1.27 1.27)) hide)
     )
@@
   (symbol (lib_id "power:+3.3V") (at 138.43 64.77 0) (unit 1)
     (in_bom yes) (on_board yes) (fields_autoplaced)
-    (property "Reference" "#PWR035" (id 0) (at 138.43 68.58 0)
+    (property "Reference" "#PWR034" (id 0) (at 138.43 68.58 0)
       (effects (font (size 1.27 1.27)) hide)
     )
@@
   (symbol (lib_id "power:GND") (at 138.43 106.68 0) (unit 1)
     (in_bom yes) (on_board yes) (fields_autoplaced)
-    (property "Reference" "#PWR036" (id 0) (at 138.43 113.03 0)
+    (property "Reference" "#PWR035" (id 0) (at 138.43 113.03 0)
       (effects (font (size 1.27 1.27)) hide)
     )
@@
   (symbol (lib_id "power:GND") (at 99.06 38.1 0) (unit 1)
     (in_bom yes) (on_board yes) (fields_autoplaced)
-    (property "Reference" "#PWR034" (id 0) (at 99.06 44.45 0)
-      (effects (font (size 1.27 1.27)) hide)
-    )
+    (property "Reference" "#PWR033" (id 0) (at 99.06 44.45 0)
+      (effects (font (size 1.27 1.27)) hide)
+    )

Commit message: Add polyfuse, 3.3V status LED, USB_CONN sheet
Parts:
- renumbered C14 to C12, C15 to C13
Changed lines of the file:
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@@
   (symbol (lib_id "power:+3.3V") (at 99.06 30.48 0) (unit 1)
     (in_bom yes) (on_board yes) (fields_autoplaced)
-    (property "Reference" "#PWR032" (id 0) (at 99.06 34.29 0)
+    (property "Reference" "#PWR028" (id 0) (at 99.06 34.29 0)
       (effects (font (size 1.27 1.27)) hide)
     )
@@
   (symbol (lib_id "power:+3.3V") (at 138.43 64.77 0) (unit 1)
     (in_bom yes) (on_board yes) (fields_autoplaced)
-    (property "Reference" "#PWR034" (id 0) (at 138.43 68.58 0)
+    (property "Reference" "#PWR030" (id 0) (at 138.43 68.58 0)
       (effects (font (size 1.27 1.27)) hide)
     )
@@
   (symbol (lib_id "Device:C") (at 105.41 34.29 0) (unit 1)
     (in_bom yes) (on_board yes) (fields_autoplaced)
-    (property "Reference" "C15" (id 0) (at 109.22 33.0199 0)
+    (property "Reference" "C13" (id 0) (at 109.22 33.0199 0)
       (effects (font (size 1.27 1.27)) (justify left))
     )
@@
   (symbol (lib_id "Device:C") (at 91.44 34.29 0) (unit 1)
     (in_bom yes) (on_board yes) (fields_autoplaced)
-    (property "Reference" "C14" (id 0) (at 95.25 33.0199 0)
+    (property "Reference" "C12" (id 0) (at 95.25 33.0199 0)
       (effects (font (size 1.27 1.27)) (justify left))
     )
@@
   (symbol (lib_id "power:GND") (at 138.43 106.68 0) (unit 1)
     (in_bom yes) (on_board yes) (fields_autoplaced)
-    (property "Reference" "#PWR035" (id 0) (at 138.43 113.03 0)
+    (property "Reference" "#PWR031" (id 0) (at 138.43 113.03 0)
       (effects (font (size 1.27 1.27)) hide)
     )
@@
   (symbol (lib_id "power:GND") (at 99.06 38.1 0) (unit 1)
     (in_bom yes) (on_board yes) (fields_autoplaced)
-    (property "Reference" "#PWR033" (id 0) (at 99.06 44.45 0)
+    (property "Reference" "#PWR029" (id 0) (at 99.06 44.45 0)
       (effects (font (size 1.27 1.27)) hide)
     )

Commit message: Fix ILI9341 display symbol (pin numbering)
Connections:
- net +3V3: now also U3.1 (VDD); no longer U3.14 (VDD)
- net DISP.BCKL: now also U3.8 (D_LED); no longer U3.7 (D_LED)
- net DISP.DC: now also U3.5 (D_DC); no longer U3.10 (D_DC)
- net DISP.RST: now also U3.4 (D_RST); no longer U3.11 (D_RST)
- net DISP.SPI_CLK: now also U3.7 (D_CLK); no longer U3.8 (D_CLK)
- net DISP.SPI_CS: now also U3.3 (D_CS); no longer U3.12 (D_CS)
- net DISP.SPI_MISO: now also R23.1; no longer R23.2
- net GND: now also U3.2 (GND); no longer U3.13 (GND)
- net TOUCH.SPI_CLK: now also U3.10 (T_CLK); no longer U3.5 (T_CLK)
- net TOUCH.SPI_CS: now also U3.11 (T_CS); no longer U3.4 (T_CS)
- net TOUCH.SPI_MOSI: now also U3.12 (T_MOSI); no longer U3.3 (T_MOSI)
- net at R21.1: now also U3.14 (T_IRQ); no longer U3.1 (T_IRQ)
- net at R22.1: now also U3.13 (T_MISO); no longer U3.2 (T_MISO)
- net at U3.9 (D_MISO): now also R23.2; no longer R23.1
Changed lines of the file:
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@@
+    (stroke (width 0) (type default) (color 0 0 0 0))
+  )
+  (wire (pts (xy 85.09 85.09) (xy 108.585 85.09))
+    (stroke (width 0) (type default) (color 0 0 0 0))
+  )
+  (wire (pts (xy 116.205 85.09) (xy 121.92 85.09))
     (stroke (width 0) (type default) (color 0 0 0 0))
   )
@@
     (stroke (width 0) (type default) (color 0 0 0 0))
   )
-  (wire (pts (xy 116.205 92.71) (xy 121.92 92.71))
+  (wire (pts (xy 85.09 92.71) (xy 121.92 92.71))
     (stroke (width 0) (type default) (color 0 0 0 0))
   )
@@
     (stroke (width 0) (type default) (color 0 0 0 0))
   )
-  (wire (pts (xy 85.09 92.71) (xy 108.585 92.71))
-    (stroke (width 0) (type default) (color 0 0 0 0))
-  )
   (wire (pts (xy 99.06 38.1) (xy 105.41 38.1))
     (stroke (width 0) (type default) (color 0 0 0 0))
@@
     (stroke (width 0) (type default) (color 0 0 0 0))
   )
-  (wire (pts (xy 85.09 85.09) (xy 121.92 85.09))
-    (stroke (width 0) (type default) (color 0 0 0 0))
-  )
   (bus (pts (xy 39.37 46.99) (xy 39.37 49.53))
     (stroke (width 0) (type default) (color 0 0 0 0))
@@
     (effects (font (size 1.27 1.27)) (justify right bottom))
   )
-  (label "DISP.SPI_MOSI" (at 85.09 85.09 0)
-    (effects (font (size 1.27 1.27)) (justify left bottom))
-  )
   (label "DISP.BCKL" (at 85.09 87.63 0)
     (effects (font (size 1.27 1.27)) (justify left bottom))
   )
+  (label "DISP.SPI_MISO" (at 85.09 85.09 0)
+    (effects (font (size 1.27 1.27)) (justify left bottom))
+  )
   (label "DISP.RST" (at 58.42 38.1 180)
     (effects (font (size 1.27 1.27)) (justify right bottom))
@@
     (effects (font (size 1.27 1.27)) (justify right bottom))
   )
+  (label "DISP.SPI_MOSI" (at 85.09 92.71 0)
+    (effects (font (size 1.27 1.27)) (justify left bottom))
+  )
   (label "TOUCH.SPI_MOSI" (at 85.09 77.47 0)
     (effects (font (size 1.27 1.27)) (justify left bottom))
@@
   (label "DISP.SPI_CS" (at 58.42 33.02 180)
     (effects (font (size 1.27 1.27)) (justify right bottom))
-  )
-  (label "DISP.SPI_MISO" (at 85.09 92.71 0)
-    (effects (font (size 1.27 1.27)) (justify left bottom))
   )
   (hierarchical_label "DISP{DISP_CONN}" (shape bidirectional) (at 35.56 20.32 180)
@@
     (pin "9")
   )
-  (symbol (lib_id "Device:R") (at 112.395 92.71 270) (mirror x) (unit 1)
-    (in_bom yes) (on_board yes)
-    (property "Reference" "R23" (id 0) (at 107.315 92.075 90))
-    (property "Value" "30" (id 1) (at 117.475 92.075 90))
-    (property "Footprint" "Resistor_SMD:R_0603_1608Metric_Pad0.98x0.95mm_HandSolder" (id 2) (at 112.395 94.488 90)
-      (effects (font (size 1.27 1.27)) hide)
-    )
-    (property "Datasheet" "~" (id 3) (at 112.395 92.71 0)
-      (effects (font (size 1.27 1.27)) hide)
-    )
-    (pin "1")
-    (pin "2")
-  )
   (symbol (lib_id "Device:R") (at 112.395 74.93 270) (mirror x) (unit 1)
     (in_bom yes) (on_board yes)
@@
       (effects (font (size 1.27 1.27)) hide)
     )
+    (pin "1")
+    (pin "2")
+  )
+  (symbol (lib_id "Device:R") (at 112.395 85.09 90) (unit 1)
+    (in_bom yes) (on_board yes)
+    (property "Reference" "R23" (id 0) (at 106.68 84.455 90))
+    (property "Value" "30" (id 1) (at 117.475 84.455 90))
+    (property "Footprint" "Resistor_SMD:R_0603_1608Metric_Pad0.98x0.95mm_HandSolder" (id 2) (at 112.395 86.868 90)
+      (effects (font (size 1.27 1.27)) hide)
+    )
+    (property "Datasheet" "~" (id 3) (at 112.395 85.09 0)
+      (effects (font (size 1.27 1.27)) hide)
+    )
