File: Board/USB_CONN.kicad_sch (KiCad schematic)
At the start: 6 parts, among them J2 USB_B_Micro

Commit message: Add I2C pin header
Parts:
- renumbered J2 to J3, R24 to R26
Changed lines of the file:
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@@
   (symbol (lib_id "Connector:USB_B_Micro") (at 105.41 69.215 0) (unit 1)
     (in_bom yes) (on_board yes)
-    (property "Reference" "J2" (id 0) (at 106.8578 57.3532 0))
+    (property "Reference" "J3" (id 0) (at 106.8578 57.3532 0))
     (property "Value" "USB_B_Micro" (id 1) (at 106.8578 59.6646 0))
     (property "Footprint" "myLib:USB_Micro-B_Molex-105017-0001" (id 2) (at 109.22 70.485 0)
@@
   (symbol (lib_id "power:+5V") (at 158.75 64.135 0) (unit 1)
     (in_bom yes) (on_board yes) (fields_autoplaced)
-    (property "Reference" "#PWR036" (id 0) (at 158.75 67.945 0)
+    (property "Reference" "#PWR039" (id 0) (at 158.75 67.945 0)
       (effects (font (size 1.27 1.27)) hide)
     )
@@
   (symbol (lib_id "power:GND") (at 134.62 71.755 0) (unit 1)
     (in_bom yes) (on_board yes)
-    (property "Reference" "#PWR034" (id 0) (at 134.62 78.105 0)
+    (property "Reference" "#PWR037" (id 0) (at 134.62 78.105 0)
       (effects (font (size 1.27 1.27)) hide)
     )
@@
   (symbol (lib_id "power:GND") (at 150.495 71.755 0) (unit 1)
     (in_bom yes) (on_board yes)
-    (property "Reference" "#PWR035" (id 0) (at 150.495 78.105 0)
+    (property "Reference" "#PWR038" (id 0) (at 150.495 78.105 0)
       (effects (font (size 1.27 1.27)) hide)
     )
@@
   (symbol (lib_id "Device:R") (at 92.71 92.71 0) (unit 1)
     (in_bom yes) (on_board yes)
-    (property "Reference" "R24" (id 0) (at 94.488 91.5416 0)
+    (property "Reference" "R26" (id 0) (at 94.488 91.5416 0)
       (effects (font (size 1.27 1.27)) (justify left))
     )
@@
   (symbol (lib_id "power:GND") (at 96.52 99.06 0) (unit 1)
     (in_bom yes) (on_board yes)
-    (property "Reference" "#PWR032" (id 0) (at 96.52 105.41 0)
+    (property "Reference" "#PWR035" (id 0) (at 96.52 105.41 0)
       (effects (font (size 1.27 1.27)) hide)
     )
@@
   (symbol (lib_id "power:GND") (at 105.41 79.375 0) (unit 1)
     (in_bom yes) (on_board yes)
-    (property "Reference" "#PWR033" (id 0) (at 105.41 85.725 0)
+    (property "Reference" "#PWR036" (id 0) (at 105.41 85.725 0)
       (effects (font (size 1.27 1.27)) hide)
     )

Commit message: Fix USB silkscreen over board warning, other minimal fixes
Changed lines of the file:
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@@
   (title_block
     (title "USB connector")
-    (date "2022/01/12")
+    (date "2022/01/17")
     (rev "v0.1")
     (company "Bzgec")
@@
     (effects (font (size 1.27 1.27)) (justify left bottom))
   )
-  (hierarchical_label "USB_N" (shape input) (at 114.3 71.755 0)
+  (hierarchical_label "USB_N" (shape bidirectional) (at 114.3 71.755 0)
     (effects (font (size 1.27 1.27)) (justify left))
   )
-  (hierarchical_label "USB_P" (shape input) (at 114.3 69.215 0)
+  (hierarchical_label "USB_P" (shape bidirectional) (at 114.3 69.215 0)
     (effects (font (size 1.27 1.27)) (justify left))
   )

Commit message: Add fiducials
Parts:
- renumbered R26 to R28
Changed lines of the file:
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@@
   (title_block
     (title "USB connector")
-    (date "2022/01/17")
+    (date "2022/01/18")
     (rev "v0.1")
     (company "Bzgec")
@@
   (symbol (lib_id "Device:R") (at 92.71 92.71 0) (unit 1)
     (in_bom yes) (on_board yes)
-    (property "Reference" "R26" (id 0) (at 94.488 91.5416 0)
-      (effects (font (size 1.27 1.27)) (justify left))
-    )
+    (property "Reference" "R28" (id 0) (at 94.488 91.5416 0)
+      (effects (font (size 1.27 1.27)) (justify left))
+    )
