File: Board/pwr.kicad_sch (KiCad schematic)
At the start: 15 parts, among them U2 MAX1821

Commit message: Add I2C pin header
Parts:
- renumbered R17 to R19, R18 to R20, R19 to R21, R20 to R22
Changed lines of the file:
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@@
   (symbol (lib_id "power:GND") (at 99.06 115.57 0) (unit 1)
     (in_bom yes) (on_board yes)
-    (property "Reference" "#PWR020" (id 0) (at 99.06 121.92 0)
+    (property "Reference" "#PWR023" (id 0) (at 99.06 121.92 0)
       (effects (font (size 1.27 1.27)) hide)
     )
@@
   (symbol (lib_id "power:GND") (at 105.41 115.57 0) (unit 1)
     (in_bom yes) (on_board yes)
-    (property "Reference" "#PWR021" (id 0) (at 105.41 121.92 0)
+    (property "Reference" "#PWR024" (id 0) (at 105.41 121.92 0)
       (effects (font (size 1.27 1.27)) hide)
     )
@@
   (symbol (lib_id "Device:R") (at 124.46 111.76 0) (unit 1)
     (in_bom yes) (on_board yes)
-    (property "Reference" "R17" (id 0) (at 126.238 110.5916 0)
+    (property "Reference" "R19" (id 0) (at 126.238 110.5916 0)
       (effects (font (size 1.27 1.27)) (justify left))
     )
@@
   (symbol (lib_id "power:GND") (at 77.47 116.84 0) (unit 1)
     (in_bom yes) (on_board yes)
-    (property "Reference" "#PWR018" (id 0) (at 77.47 123.19 0)
+    (property "Reference" "#PWR021" (id 0) (at 77.47 123.19 0)
       (effects (font (size 1.27 1.27)) hide)
     )
@@
   (symbol (lib_id "power:GND") (at 124.46 123.19 0) (unit 1)
     (in_bom yes) (on_board yes)
-    (property "Reference" "#PWR022" (id 0) (at 124.46 129.54 0)
+    (property "Reference" "#PWR025" (id 0) (at 124.46 129.54 0)
       (effects (font (size 1.27 1.27)) hide)
     )
@@
   (symbol (lib_id "Device:R") (at 152.4 92.71 0) (unit 1)
     (in_bom yes) (on_board yes)
-    (property "Reference" "R18" (id 0) (at 154.178 91.5416 0)
+    (property "Reference" "R20" (id 0) (at 154.178 91.5416 0)
       (effects (font (size 1.27 1.27)) (justify left))
     )
@@
   (symbol (lib_id "Device:R") (at 152.4 100.33 0) (unit 1)
     (in_bom yes) (on_board yes)
-    (property "Reference" "R19" (id 0) (at 154.178 99.1616 0)
+    (property "Reference" "R21" (id 0) (at 154.178 99.1616 0)
       (effects (font (size 1.27 1.27)) (justify left))
     )
@@
   (symbol (lib_id "power:GND") (at 152.4 104.14 0) (unit 1)
     (in_bom yes) (on_board yes)
-    (property "Reference" "#PWR024" (id 0) (at 152.4 110.49 0)
+    (property "Reference" "#PWR027" (id 0) (at 152.4 110.49 0)
       (effects (font (size 1.27 1.27)) hide)
     )
@@
   (symbol (lib_id "power:GND") (at 86.36 96.52 0) (unit 1)
     (in_bom yes) (on_board yes)
-    (property "Reference" "#PWR019" (id 0) (at 86.36 102.87 0)
+    (property "Reference" "#PWR022" (id 0) (at 86.36 102.87 0)
       (effects (font (size 1.27 1.27)) hide)
     )
@@
   (symbol (lib_id "power:+5V") (at 55.88 80.01 0) (unit 1)
     (in_bom yes) (on_board yes) (fields_autoplaced)
-    (property "Reference" "#PWR015" (id 0) (at 55.88 83.82 0)
+    (property "Reference" "#PWR018" (id 0) (at 55.88 83.82 0)
       (effects (font (size 1.27 1.27)) hide)
     )
@@
   (symbol (lib_id "power:+3.3V") (at 189.23 80.01 0) (unit 1)
     (in_bom yes) (on_board yes) (fields_autoplaced)
-    (property "Reference" "#PWR026" (id 0) (at 189.23 83.82 0)
+    (property "Reference" "#PWR029" (id 0) (at 189.23 83.82 0)
       (effects (font (size 1.27 1.27)) hide)
     )
@@
   (symbol (lib_id "power:GNDPWR") (at 69.85 88.9 0) (unit 1)
     (in_bom yes) (on_board yes) (fields_autoplaced)
-    (property "Reference" "#PWR017" (id 0) (at 69.85 93.98 0)
+    (property "Reference" "#PWR020" (id 0) (at 69.85 93.98 0)
       (effects (font (size 1.27 1.27)) hide)
     )
@@
   (symbol (lib_id "Device:R") (at 189.23 101.6 0) (unit 1)
     (in_bom yes) (on_board yes) (fields_autoplaced)
-    (property "Reference" "R20" (id 0) (at 191.77 100.3299 0)
+    (property "Reference" "R22" (id 0) (at 191.77 100.3299 0)
       (effects (font (size 1.27 1.27)) (justify left))
     )
@@
   (symbol (lib_id "power:GND") (at 169.545 87.63 0) (unit 1)
     (in_bom yes) (on_board yes) (fields_autoplaced)
-    (property "Reference" "#PWR025" (id 0) (at 169.545 93.98 0)
+    (property "Reference" "#PWR028" (id 0) (at 169.545 93.98 0)
       (effects (font (size 1.27 1.27)) hide)
     )
@@
   (symbol (lib_id "power:GND") (at 189.23 105.41 0) (unit 1)
     (in_bom yes) (on_board yes) (fields_autoplaced)
-    (property "Reference" "#PWR027" (id 0) (at 189.23 111.76 0)
+    (property "Reference" "#PWR030" (id 0) (at 189.23 111.76 0)
       (effects (font (size 1.27 1.27)) hide)
     )
@@
   (symbol (lib_id "power:GNDPWR") (at 49.53 180.34 0) (unit 1)
     (in_bom yes) (on_board yes) (fields_autoplaced)
-    (property "Reference" "#PWR014" (id 0) (at 49.53 185.42 0)
+    (property "Reference" "#PWR017" (id 0) (at 49.53 185.42 0)
       (effects (font (size 1.27 1.27)) hide)
     )
@@
   (symbol (lib_id "power:GND") (at 58.42 180.34 0) (unit 1)
     (in_bom yes) (on_board yes) (fields_autoplaced)
-    (property "Reference" "#PWR016" (id 0) (at 58.42 186.69 0)
+    (property "Reference" "#PWR019" (id 0) (at 58.42 186.69 0)
       (effects (font (size 1.27 1.27)) hide)
     )
@@
   (symbol (lib_id "power:GNDPWR") (at 130.81 87.63 0) (unit 1)
     (in_bom yes) (on_board yes) (fields_autoplaced)
-    (property "Reference" "#PWR023" (id 0) (at 130.81 92.71 0)
-      (effects (font (size 1.27 1.27)) hide)
-    )
+    (property "Reference" "#PWR026" (id 0) (at 130.81 92.71 0)
+      (effects (font (size 1.27 1.27)) hide)
+    )

Commit message: Add fiducials
Parts:
- renumbered R19 to R21, R20 to R22, R21 to R23, R22 to R24
Changed lines of the file:
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@@
   (title_block
     (title "Power supply")
-    (date "2022/01/17")
+    (date "2022/01/18")
     (rev "v0.1")
     (company "Bzgec")
@@
   (symbol (lib_id "Device:R") (at 124.46 111.76 0) (unit 1)
     (in_bom yes) (on_board yes)
-    (property "Reference" "R19" (id 0) (at 126.238 110.5916 0)
+    (property "Reference" "R21" (id 0) (at 126.238 110.5916 0)
       (effects (font (size 1.27 1.27)) (justify left))
     )
@@
   (symbol (lib_id "Device:R") (at 152.4 92.71 0) (unit 1)
     (in_bom yes) (on_board yes)
-    (property "Reference" "R20" (id 0) (at 154.178 91.5416 0)
+    (property "Reference" "R22" (id 0) (at 154.178 91.5416 0)
       (effects (font (size 1.27 1.27)) (justify left))
     )
@@
   (symbol (lib_id "Device:R") (at 152.4 100.33 0) (unit 1)
     (in_bom yes) (on_board yes)
-    (property "Reference" "R21" (id 0) (at 154.178 99.1616 0)
+    (property "Reference" "R23" (id 0) (at 154.178 99.1616 0)
       (effects (font (size 1.27 1.27)) (justify left))
     )
@@
   (symbol (lib_id "Device:R") (at 189.23 101.6 0) (unit 1)
     (in_bom yes) (on_board yes) (fields_autoplaced)
-    (property "Reference" "R22" (id 0) (at 191.77 100.3299 0)
-      (effects (font (size 1.27 1.27)) (justify left))
-    )
+    (property "Reference" "R24" (id 0) (at 191.77 100.3299 0)
+      (effects (font (size 1.27 1.27)) (justify left))
+    )

Commit message: Fix buck inductor (uF -> uH)
Parts:
- L1: value 10uF -> 10uH
Changed lines of the file:
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@@
     (in_bom yes) (on_board yes)
     (property "Reference" "L1" (id 0) (at 123.19 75.184 90))
-    (property "Value" "10uF" (id 1) (at 123.19 77.4954 90))
+    (property "Value" "10uH" (id 1) (at 123.19 77.4954 90))
     (property "Footprint" "myLib:NR6028T100M" (id 2) (at 123.19 80.01 0)
       (effects (font (size 1.27 1.27)) hide)
